File: QCM_driver/QCM_driver.kicad_sch (KiCad schematic)
At the start: 86 parts, among them J1 Conn_Coaxial, J2 Conn_Coaxial, J3 Conn_Coaxial, J4 Conn_Coaxial, J5 Conn_Coaxial, J6 Conn_Coaxial, U1 OPA656U, U2 OPA656U, U3 OPA656U, U4 AD835ARZ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

Commit message: PCB and schematic V1.0
Parts:
- R24, R26, R30, R31, R32, R34: value 0 -> DNP
Other:
- sheet VCO IC B 1 renamed VCO IC 1
- sheet VCO IC B 2 renamed VCO IC 2
- sheet VCO IC 1: file VCO_B.kicad_sch -> VCO_IC.kicad_sch
- sheet VCO IC 2: file VCO_B.kicad_sch -> VCO_IC.kicad_sch
- note added: "Loop Filter"
- note removed: "Integrate"
Changed lines of the file:
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@@
   )
   (polyline (pts (xy 86.36 68.58) (xy 86.36 240.03))
-    (stroke (width 0) (type default))
+    (stroke (width 0) (type dash))
   )
   (wire (pts (xy 344.17 203.2) (xy 354.33 203.2))
@@
   )
   (polyline (pts (xy 257.81 71.12) (xy 257.81 241.3))
-    (stroke (width 0) (type default))
+    (stroke (width 0) (type dash))
   )
   (wire (pts (xy 156.21 187.96) (xy 171.45 187.96))
@@
   )
   (polyline (pts (xy 166.37 71.12) (xy 166.37 241.3))
-    (stroke (width 0) (type default))
+    (stroke (width 0) (type dash))
   )
   (wire (pts (xy 356.87 217.17) (xy 359.41 217.17))
@@
   )
   (polyline (pts (xy 339.09 73.66) (xy 339.09 242.57))
-    (stroke (width 0) (type default))
+    (stroke (width 0) (type dash))
   )
   (wire (pts (xy 181.61 134.62) (xy 171.45 134.62))
@@
   )
   (polyline (pts (xy 220.98 71.12) (xy 220.98 241.3))
-    (stroke (width 0) (type default))
+    (stroke (width 0) (type dash))
   )
   (wire (pts (xy 257.81 50.8) (xy 262.89 50.8))
@@
     (effects (font (size 1.27 1.27)) (justify left bottom))
   )
-  (text "Integrate" (at 302.26 80.01 0)
+  (text "Loop Filter" (at 294.64 80.01 0)
     (effects (font (size 1.27 1.27)) (justify left bottom))
   )
@@
       (effects (font (size 1.27 1.27)))
     )
-    (property "Value" "0" (at 363.22 217.17 90)
+    (property "Value" "DNP" (at 363.22 217.17 90)
       (effects (font (size 1.27 1.27)))
     )
@@
       (effects (font (size 1.27 1.27)))
     )
-    (property "Value" "0" (at 349.25 182.88 90)
+    (property "Value" "DNP" (at 349.25 182.88 90)
       (effects (font (size 1.27 1.27)))
     )
@@
       (effects (font (size 1.27 1.27)))
     )
-    (property "Value" "0" (at 384.81 180.34 90)
+    (property "Value" "DNP" (at 384.81 180.34 90)
       (effects (font (size 1.27 1.27)))
     )
@@
       (effects (font (size 1.27 1.27)))
     )
-    (property "Value" "0" (at 384.81 119.38 90)
+    (property "Value" "DNP" (at 384.81 119.38 90)
       (effects (font (size 1.27 1.27)))
     )
@@
       (effects (font (size 1.27 1.27)))
     )
-    (property "Value" "0" (at 363.22 156.21 90)
+    (property "Value" "DNP" (at 363.22 156.21 90)
       (effects (font (size 1.27 1.27)))
     )
@@
       (effects (font (size 1.27 1.27)))
     )
-    (property "Value" "0" (at 349.25 121.92 90)
+    (property "Value" "DNP" (at 349.25 121.92 90)
       (effects (font (size 1.27 1.27)))
     )
@@
     (stroke (width 0.1524) (type solid))
     (fill (color 0 0 0 0.0000))
-    (property "Sheetname" "VCO IC B 2" (at 354.33 193.5984 0)
+    (property "Sheetname" "VCO IC 2" (at 354.33 193.5984 0)
       (effects (font (size 1.27 1.27)) (justify left bottom))
     )
-    (property "Sheetfile" "VCO_B.kicad_sch" (at 354.33 207.5946 0)
+    (property "Sheetfile" "VCO_IC.kicad_sch" (at 354.33 207.5946 0)
       (effects (font (size 1.27 1.27)) (justify left top))
     )
@@
     (stroke (width 0.1524) (type solid))
     (fill (color 0 0 0 0.0000))
-    (property "Sheetname" "VCO IC B 1" (at 354.33 132.6384 0)
+    (property "Sheetname" "VCO IC 1" (at 354.33 132.6384 0)
       (effects (font (size 1.27 1.27)) (justify left bottom))
     )
-    (property "Sheetfile" "VCO_B.kicad_sch" (at 354.33 146.6346 0)
+    (property "Sheetfile" "VCO_IC.kicad_sch" (at 354.33 146.6346 0)
       (effects (font (size 1.27 1.27)) (justify left top))
     )
